File: Audio and Video.sch (KiCad schematic (older format))
At the start: 37 parts, among them J106 pin, J107 pin, Q10 PN2222A, Q11 PN2222A, U1 LM358, U19 LM555

Commit message: SMD Audio
Parts:
- removed C20: 4,7uF, Capacitor_THT:C_Rect_L7.2mm_W7.2mm_P5.00mm_FKS2_FKP2_MKS2_MKP2, symbol Device:C
- removed C23: 47nF, Atari:C_Axial_L5.1mm_D2.5mm_P12.50mm_Horizontal, symbol Device:C
- removed C24: 10uF, Capacitor_THT:CP_Radial_D7.5mm_P2.50mm, symbol Device:CP
- removed J106, J107: pin, Connector_PinHeader_2.00mm:PinHeader_1x01_P2.00mm_Vertical, symbol Connector_Generic:Conn_01x01
- removed R1, R11: 2k2, Atari:R_Axial_DIN0207_L3.6mm_D2.2mm_P10.16mm_Horizontal, symbol Device:R
- removed R3: 6k2, Atari:R_Axial_DIN0207_L3.6mm_D2.2mm_P10.16mm_Horizontal, symbol Device:R
- removed R4: 56k, Atari:R_Axial_DIN0207_L3.6mm_D2.2mm_P10.16mm_Horizontal, symbol Device:R
- removed U1: LM358, Package_DIP:DIP-8_W7.62mm_Socket, symbol Amplifier_Operational:LM358
- added Q101: BC849, Package_TO_SOT_SMD:SOT-23, symbol Transistor_BJT:BC849
- C112, C16, C21: value 1nF -> 100nF; footprint Atari:C_Axial_L5.1mm_D2.5mm_P12.50mm_Horizontal -> Capacitor_SMD:C_1206_3216Metric_Pad1.42x1.75mm_HandSolder
- C17: value 47nF -> 100nF; footprint Atari:C_Axial_L5.1mm_D2.5mm_P12.50mm_Horizontal -> Capacitor_SMD:C_1206_3216Metric_Pad1.42x1.75mm_HandSolder
- C19: value 4,7uF -> 10uF; footprint Capacitor_THT:C_Rect_L7.2mm_W7.2mm_P5.00mm_FKS2_FKP2_MKS2_MKP2 -> Capacitor_SMD:C_1210_3225Metric_Pad1.42x2.65mm_HandSolder
- C22: value 4,7uF -> 100nF; footprint Capacitor_THT:C_Rect_L7.2mm_W7.2mm_P5.00mm_FKS2_FKP2_MKS2_MKP2 -> Capacitor_SMD:C_1206_3216Metric_Pad1.42x1.75mm_HandSolder
- R10: value 1k -> 15k; footprint Atari:R_Axial_DIN0207_L3.6mm_D2.2mm_P10.16mm_Horizontal -> Resistor_SMD:R_1206_3216Metric_Pad1.42x1.75mm_HandSolder
- R2: value 1k -> 10; footprint Atari:R_Axial_DIN0207_L3.6mm_D2.2mm_P10.16mm_Horizontal -> Resistor_SMD:R_1206_3216Metric_Pad1.42x1.75mm_HandSolder
- R5: value 470k -> 100k; footprint Atari:R_Axial_DIN0207_L3.6mm_D2.2mm_P10.16mm_Horizontal -> Resistor_SMD:R_1206_3216Metric_Pad1.42x1.75mm_HandSolder
- R6: value 68k -> 100k; footprint Atari:R_Axial_DIN0207_L3.6mm_D2.2mm_P10.16mm_Horizontal -> Resistor_SMD:R_1206_3216Metric_Pad1.42x1.75mm_HandSolder
- R7: value 2k -> 100k; footprint Atari:R_Axial_DIN0207_L3.6mm_D2.2mm_P10.16mm_Horizontal -> Resistor_SMD:R_1206_3216Metric_Pad1.42x1.75mm_HandSolder
- R8: value 5k1 -> 470k; footprint Atari:R_Axial_DIN0207_L3.6mm_D2.2mm_P10.16mm_Horizontal -> Resistor_SMD:R_1206_3216Metric_Pad1.42x1.75mm_HandSolder
- R9: value 3k3 -> 470k; footprint Atari:R_Axial_DIN0207_L3.6mm_D2.2mm_P10.16mm_Horizontal -> Resistor_SMD:R_1206_3216Metric_Pad1.42x1.75mm_HandSolder
Connections:
- wire segments 100 -> 62
Other:
- moved on the sheet: C112, C16, C17, C19, C200, C201, C21, C22, L14, R10, R2, R200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

Commit message: Almost finished
Connections:
- net COMPOSITE_A renamed COMPOSITE
Changed lines of the file:
@@
 	4500 6250 4500 6325
 Text GLabel 4925 6250 2    50   Input ~ 0
-COMPOSITE_A
+COMPOSITE
 Text GLabel 1900 3075 0    50   Input ~ 0
 EXTAUDIO
