File: Power.sch (KiCad schematic (older format))
At the start: 33 parts, among them J11 C, J12 C, J13 C, J14 C, J15 C, J16 C, J17 C, J18 C, J19 C, J20 C, J21 C, J7 Power, SW1 Switch_power_on

Commit message: SMD power
Parts:
- removed C205: 100nF, Atari:C_Axial_L5.1mm_D2.5mm_P12.50mm_Horizontal, symbol Device:C
- removed J11, J12, J13, J14, J15, J16, J17, J18, J19, J20, J21: C, Connector_PinHeader_2.54mm:PinHeader_1x01_P2.54mm_Vertical, symbol Connector_Generic:Conn_01x01
- removed L13: 820uH, Atari:L_Axial_L7.0mm_D3.3mm_P12.50mm_Horizontal_Fastron_MICC, symbol Device:L
- C1: footprint Capacitor_THT:CP_Radial_D8.0mm_P3.80mm -> Capacitor_SMD:CP_Elec_10x10.5
- C10, C2, C3: footprint Capacitor_THT:CP_Radial_D7.5mm_P2.50mm -> Capacitor_SMD:CP_Elec_6.3x5.2
- C11, C12, C13, C14, C15, C4, C5, C6, C7, C8, C9: footprint Atari:C_Axial_L5.1mm_D2.5mm_P12.50mm_Horizontal -> Capacitor_SMD:C_1206_3216Metric_Pad1.42x1.75mm_HandSolder
- FB1, FB2, FB3: footprint Atari:L_Axial_L7.0mm_D3.3mm_P12.50mm_Horizontal_Fastron_MICC -> Inductor_SMD:L_1812_4532Metric_Pad1.30x3.40mm_HandSolder
