File: Atari 130XE 1MB smd.kicad_pcb (KiCad board)
At the start: 2 copper layers, 324 x 204 mm, 379 parts, among them J1 SIO, J10 Mem_on_off, J102 pin, J103 pin, J104 pin, J105 pin, J106 pin, J107 pin, J2 Video, J201 Diagnostic, J202 Diag, J210 Diag, J24 Cartridge, J4 Expansion, J5 Joystick_Port, J50 Test_signal, J500 Basic_sel, J501 TPP_sel, J51 To_GND, J6 Joystick_Port, J7 Power, J8 Keyboard, Q1 2N3904, Q10 PN2222A, Q11 PN2222A, Q2 2N3904, Q3 2N3904, Q4 2N3906, Q6 2N3904, SW1 Switch_power_on, U1 LM358, U10 DRAM_4464, U100 74LS157, U101 74LS74, U102 74HC02, U103 74HC02, U104 74LS157, U105 74LVC2G74, U17 GTIA, U18 74LS08, U19 LM555, U2 74LS138, U20 4050, U21 74LS74, U22 POKEY, U23 PIA, U24 CD4051B, U25 CD4051B, U3 MMU, U4 27C010, U40 GAL20V8_DIP, U41 74LS157, U42 74LS175, U43 DRAM_1MB_4bit, U44 DRAM_1MB_4bit, U5 27C010, U6 Freddie, U7 Antic, U8 Sally, U9 DRAM_4464, Y1 Crystal, Y2 4,43 MHz

Commit message: SMD Audio
Parts:
- removed C20: 4,7uF, Capacitor_THT:C_Rect_L7.2mm_W7.2mm_P5.00mm_FKS2_FKP2_MKS2_MKP2
- removed C23: 47nF, Atari:C_Axial_L5.1mm_D2.5mm_P12.50mm_Horizontal
- removed C24: 10uF, Capacitor_THT:CP_Radial_D7.5mm_P2.50mm
- removed J106, J107: pin, Connector_PinHeader_2.00mm:PinHeader_1x01_P2.00mm_Vertical
- removed R1, R11: 2k2, Atari:R_Axial_DIN0207_L3.6mm_D2.2mm_P10.16mm_Horizontal
- removed R3: 6k2, Atari:R_Axial_DIN0207_L3.6mm_D2.2mm_P10.16mm_Horizontal
- removed R4: 56k, Atari:R_Axial_DIN0207_L3.6mm_D2.2mm_P10.16mm_Horizontal
- removed U1: LM358, Package_DIP:DIP-8_W7.62mm_Socket
- added Q101: BC849, Package_TO_SOT_SMD:SOT-23, F.Cu at (116.2, 113.7)
- C112, C16, C21: value 1nF -> 100nF; footprint Atari:C_Axial_L5.1mm_D2.5mm_P12.50mm_Horizontal -> Capacitor_SMD:C_1206_3216Metric_Pad1.42x1.75mm_HandSolder
- C17: value 47nF -> 100nF; footprint Atari:C_Axial_L5.1mm_D2.5mm_P12.50mm_Horizontal -> Capacitor_SMD:C_1206_3216Metric_Pad1.42x1.75mm_HandSolder
- C19: value 4,7uF -> 10uF; footprint Capacitor_THT:C_Rect_L7.2mm_W7.2mm_P5.00mm_FKS2_FKP2_MKS2_MKP2 -> Capacitor_SMD:C_1210_3225Metric_Pad1.42x2.65mm_HandSolder
- C22: value 4,7uF -> 100nF; footprint Capacitor_THT:C_Rect_L7.2mm_W7.2mm_P5.00mm_FKS2_FKP2_MKS2_MKP2 -> Capacitor_SMD:C_1206_3216Metric_Pad1.42x1.75mm_HandSolder
- R10: value 1k -> 15k; footprint Atari:R_Axial_DIN0207_L3.6mm_D2.2mm_P10.16mm_Horizontal -> Resistor_SMD:R_1206_3216Metric_Pad1.42x1.75mm_HandSolder
- R2: value 1k -> 10; footprint Atari:R_Axial_DIN0207_L3.6mm_D2.2mm_P10.16mm_Horizontal -> Resistor_SMD:R_1206_3216Metric_Pad1.42x1.75mm_HandSolder
- R5: value 470k -> 100k; footprint Atari:R_Axial_DIN0207_L3.6mm_D2.2mm_P10.16mm_Horizontal -> Resistor_SMD:R_1206_3216Metric_Pad1.42x1.75mm_HandSolder
- R6: value 68k -> 100k; footprint Atari:R_Axial_DIN0207_L3.6mm_D2.2mm_P10.16mm_Horizontal -> Resistor_SMD:R_1206_3216Metric_Pad1.42x1.75mm_HandSolder
- R7: value 2k -> 100k; footprint Atari:R_Axial_DIN0207_L3.6mm_D2.2mm_P10.16mm_Horizontal -> Resistor_SMD:R_1206_3216Metric_Pad1.42x1.75mm_HandSolder
- R8: value 5k1 -> 470k; footprint Atari:R_Axial_DIN0207_L3.6mm_D2.2mm_P10.16mm_Horizontal -> Resistor_SMD:R_1206_3216Metric_Pad1.42x1.75mm_HandSolder
- R9: value 3k3 -> 470k; footprint Atari:R_Axial_DIN0207_L3.6mm_D2.2mm_P10.16mm_Horizontal -> Resistor_SMD:R_1206_3216Metric_Pad1.42x1.75mm_HandSolder
- moved C22 65.2 mm to (121.9, 128.2)
- moved R5 30.2 mm to (116.9, 119.0), turned to 180 degrees
- moved R80 30.0 mm to (121.9, 130.5)
- moved C19 26.6 mm to (121.9, 113.7)
- moved C16 26.3 mm to (121.9, 121.3), turned to 180 degrees
- moved C17 25.4 mm to (121.9, 125.9)
- moved R8 23.5 mm to (116.9, 121.3), turned to 0 degrees
- moved C112 23.2 mm to (121.9, 123.6)
- moved R6 22.2 mm to (116.9, 123.6), turned to 0 degrees
- moved R10 21.3 mm to (116.9, 116.6), turned to 0 degrees
- moved R2 17.6 mm to (121.9, 119.0), turned to 0 degrees
- moved R7 15.2 mm to (116.9, 128.2), turned to 0 degrees
- moved R9 12.8 mm to (116.9, 125.9), turned to 0 degrees
- moved C21 5.44 mm to (121.9, 116.6), turned to 180 degrees
Connections:
- C112 pad 1: GND -> SIOAUDIO
- C112 pad 2: SIOAUDIO -> Net-(C112-Pad2)
- C16 pad 1: GND -> EXTAUDIO
- C16 pad 2: +5C -> Net-(C16-Pad2)
- C17 pad 2: SOUND -> BELL
- C19 pad 2: SIOAUDIO -> AUDIO
- C21 pad 2: Net-(C19-Pad1) -> Net-(C21-Pad2)
- C22 pad 1: EXTAUDIO -> SOUND
- C22 pad 2: Net-(C19-Pad1) -> Net-(C22-Pad2)
- J1 pad 12: (no net) -> Net-(J1-Pad12)
- J4 pad A: (no net) -> Net-(J4-PadA)
- R10 pad 1: AUDIO -> Net-(C19-Pad1)
- R10 pad 2: GND -> Net-(Q101-Pad1)
- R2 pad 1: Net-(C19-Pad1) -> Net-(C21-Pad2)
- R2 pad 2: Net-(R1-Pad2) -> +5C
- R5 pad 1: Net-(C23-Pad1) -> Net-(C21-Pad2)
- R5 pad 2: Net-(R5-Pad2) -> Net-(C19-Pad1)
- R6 pad 1: Net-(R6-Pad1) -> Net-(Q101-Pad1)
- R6 pad 2: Net-(R5-Pad2) -> Net-(C112-Pad2)
- R7 pad 1: Net-(R5-Pad2) -> Net-(Q101-Pad1)
- R7 pad 2: Net-(C20-Pad1) -> Net-(C22-Pad2)
- R8 pad 1: AUDIO -> Net-(Q101-Pad1)
- R8 pad 2: Net-(R6-Pad1) -> Net-(C16-Pad2)
- R9 pad 1: +5C -> Net-(Q101-Pad1)
- R9 pad 2: Net-(C24-Pad1) -> Net-(C17-Pad1)
- SW1 pad 1: (no net) -> Net-(SW1-Pad1)
- U104 pad 12: (no net) -> Net-(U104-Pad12)
- U105 pad 3: (no net) -> Net-(U105-Pad3)
- U17 pad 10: (no net) -> Net-(U17-Pad10)
- U19 pad 5: (no net) -> Net-(U19-Pad5)
- U19 pad 7: (no net) -> Net-(U19-Pad7)
- U2 pad 11: (no net) -> D4XX
- U2 pad 7: (no net) -> D7XX
- U20 pad 10: (no net) -> Net-(U20-Pad10)
- U40 pad 11: (no net) -> Net-(U40-Pad11)
- U40 pad 20: (no net) -> Net-(U40-Pad20)
- U41 pad 10: (no net) -> Net-(U41-Pad10)
- U41 pad 11: (no net) -> Net-(U41-Pad11)
- U41 pad 12: (no net) -> Net-(U41-Pad12)
- U41 pad 13: (no net) -> Net-(U41-Pad13)
- U41 pad 14: (no net) -> Net-(U41-Pad14)
- U41 pad 9: (no net) -> Net-(U41-Pad9)
- U42 pad 10: (no net) -> Net-(U42-Pad10)
- U42 pad 11: (no net) -> Net-(U42-Pad11)
- U42 pad 12: (no net) -> Net-(U42-Pad12)
- U42 pad 13: (no net) -> Net-(U42-Pad13)
- U42 pad 14: (no net) -> Net-(U42-Pad14)
- U42 pad 15: (no net) -> Net-(U42-Pad15)
- U42 pad 3: (no net) -> Net-(U42-Pad3)
- U42 pad 6: (no net) -> Net-(U42-Pad6)
- U6 pad 36: (no net) -> Net-(U6-Pad36)
- U6 pad 6: (no net) -> Net-(U6-Pad6)
- U6 pad 7: (no net) -> Net-(U6-Pad7)
- U8 pad 34: (no net) -> Net-(U8-Pad34)
- U8 pad 5: (no net) -> Net-(U8-Pad5)
- U8 pad 7: (no net) -> Net-(U8-Pad7)
Routing:
- net Net-(C19-Pad1): track 119.7 -> 10.6 mm, vias 2 -> 0
- net EXTAUDIO: track 30.6 -> 112.2 mm, vias 2 -> 5
- net Net-(C24-Pad1): track 68.5 -> 0.00 mm
- net Net-(R1-Pad1): track 54.6 -> 0.00 mm
- net Net-(R5-Pad2): track 44.4 -> 0.00 mm, vias 1 -> 0
- net Net-(C20-Pad1): track 41.9 -> 0.00 mm
- net Net-(R1-Pad2): track 38.7 -> 0.00 mm
- net Net-(R6-Pad1): track 32.9 -> 0.00 mm
- net MONO_MOD: track 64.8 -> 34.5 mm, vias 2 -> 0
- net COMPOSITE: track 32.7 -> 4.65 mm
- net SOUND: track 157.1 -> 184.8 mm
- net BELL: track 104.4 -> 130.6 mm, vias 0 -> 3
- net GND: track 1704.4 -> 1679.7 mm
- net COLOR: track 79.4 -> 56.2 mm
- net SIOAUDIO: track 269.3 -> 246.8 mm, vias 5 -> 6
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Other:
- board text removed: "LM358"

Commit message: SMD ram
Parts:
- R100, R101, R102, R103, R104, R105, R106, R107, R110, R111, R207, R208, R209, R210, R211, R212, R213, R214: footprint Atari:R_Axial_DIN0207_L3.6mm_D2.2mm_P10.16mm_Horizontal -> Resistor_SMD:R_1206_3216Metric_Pad1.42x1.75mm_HandSolder
- moved R104 38.9 mm to (105.5, 141.7), turned to 270 degrees
- moved R105 33.9 mm to (96.3, 141.7), turned to 270 degrees
- moved R103 32.5 mm to (100.9, 141.7), turned to 270 degrees
- moved R208 29.4 mm to (98.6, 141.7), turned to 270 degrees
- moved R207 26.0 mm to (93.9, 141.7), turned to 270 degrees
- moved R111 25.7 mm to (119.4, 141.7), turned to 270 degrees
- moved R100 20.9 mm to (114.7, 141.7), turned to 270 degrees
- moved R102 20.0 mm to (110.1, 141.7), turned to 270 degrees
- moved R210 19.9 mm to (107.8, 141.7), turned to 270 degrees
- moved R106 19.6 mm to (100.2, 120.4)
- moved R209 19.2 mm to (103.2, 141.7), turned to 270 degrees
- moved R211 19.0 mm to (112.5, 141.7), turned to 270 degrees
- moved R107 17.8 mm to (100.2, 115.8)
- moved R214 12.5 mm to (100.2, 113.5)
- moved R101 12.0 mm to (100.2, 125.0)
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Connections:
- J1 pad 12: Net-(J1-Pad12) -> (no net)
- J4 pad A: Net-(J4-PadA) -> (no net)
- SW1 pad 1: Net-(SW1-Pad1) -> (no net)
- U104 pad 12: Net-(U104-Pad12) -> (no net)
- U105 pad 3: Net-(U105-Pad3) -> (no net)
- U17 pad 10: Net-(U17-Pad10) -> (no net)
- U19 pad 5: Net-(U19-Pad5) -> (no net)
- U19 pad 7: Net-(U19-Pad7) -> (no net)
- U2 pad 11: D4XX -> (no net)
- U2 pad 7: D7XX -> (no net)
- U20 pad 10: Net-(U20-Pad10) -> (no net)
- U40 pad 11: Net-(U40-Pad11) -> (no net)
- U40 pad 20: Net-(U40-Pad20) -> (no net)
- U41 pad 10: Net-(U41-Pad10) -> (no net)
- U41 pad 11: Net-(U41-Pad11) -> (no net)
- U41 pad 12: Net-(U41-Pad12) -> (no net)
- U41 pad 13: Net-(U41-Pad13) -> (no net)
- U41 pad 14: Net-(U41-Pad14) -> (no net)
- U41 pad 9: Net-(U41-Pad9) -> (no net)
- U42 pad 10: Net-(U42-Pad10) -> (no net)
- U42 pad 11: Net-(U42-Pad11) -> (no net)
- U42 pad 12: Net-(U42-Pad12) -> (no net)
- U42 pad 13: Net-(U42-Pad13) -> (no net)
- U42 pad 14: Net-(U42-Pad14) -> (no net)
- U42 pad 15: Net-(U42-Pad15) -> (no net)
- U42 pad 3: Net-(U42-Pad3) -> (no net)
- U42 pad 6: Net-(U42-Pad6) -> (no net)
- U6 pad 36: Net-(U6-Pad36) -> (no net)
- U6 pad 6: Net-(U6-Pad6) -> (no net)
- U6 pad 7: Net-(U6-Pad7) -> (no net)
- U8 pad 34: Net-(U8-Pad34) -> (no net)
- U8 pad 5: Net-(U8-Pad5) -> (no net)
- U8 pad 7: Net-(U8-Pad7) -> (no net)
Routing:
- net D1: track 601.1 -> 569.8 mm, vias 10 -> 11
- net DQ1: track 80.2 -> 110.6 mm, vias 1 -> 2
- net D0: track 596.3 -> 572.0 mm, vias 10 -> 11
- net DQ4: track 53.9 -> 75.7 mm, vias 2 -> 3
- net Net-(R111-Pad1): track 63.0 -> 84.0 mm, vias 2 -> 3
- net DQ3: track 93.1 -> 113.6 mm, vias 1 -> 2
- net D2: track 603.5 -> 584.0 mm, vias 10 -> 11
- net DQ0: track 88.0 -> 106.2 mm, vias 1 -> 2
- net D7: track 478.1 -> 461.6 mm, vias 9 -> 10
- net CASMAN: track 65.3 -> 80.5 mm, vias 0 -> 1
- net D3: track 505.3 -> 490.3 mm, vias 7 -> 8
- net D5: track 490.6 -> 477.2 mm, vias 7 -> 8
- net DQ2: track 98.4 -> 111.5 mm, vias 1 -> 2
- net +5VA: track 2202.6 -> 2213.8 mm, vias 57 -> 59
- net D6: track 477.6 -> 469.4 mm, vias 7 -> 8
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
Commit message: Basic smd
Parts:
- removed R205: 150, Atari:R_Axial_DIN0207_L3.6mm_D2.2mm_P10.16mm_Horizontal
- added D1000: 1N4002, Diode_THT:D_DO-41_SOD81_P12.70mm_Horizontal, F.Cu at (137.0, 150.4)
- C42: footprint Atari:C_Axial_L5.1mm_D2.5mm_P12.50mm_Horizontal -> Capacitor_SMD:C_1206_3216Metric_Pad1.42x1.75mm_HandSolder
- C50: value 10uF -> 220uF
- R116: value 51 -> 8,2
- R202: value 180 -> 75
- R204: value 47 -> 75
- R53: value 100 -> 75
- moved R503 207.1 mm to (105.9, 56.5), turned to 0 degrees
- moved R504 206.5 mm to (105.9, 59.8), turned to 0 degrees
- moved R505 206.2 mm to (111.9, 56.5), turned to 0 degrees
- moved R506 205.6 mm to (111.9, 59.8), turned to 0 degrees
- moved J500 204.6 mm to (105.7, 64.4)
- moved J501 204.6 mm to (114.9, 66.9)
- moved R510 198.3 mm to (120.8, 63.5)
- moved C99 34.2 mm to (251.9, 209.9), turned to 270 degrees
- moved U104 31.4 mm to (258.5, 211.1), turned to 90 degrees
- moved U105 30.6 mm to (266.8, 211.9), turned to 90 degrees
- moved C203 30.4 mm to (270.0, 211.3), turned to 270 degrees
- moved D100 11.7 mm to (262.0, 202.7)
- moved R508 11.7 mm to (259.6, 202.7)
- moved U5 11.7 mm to (211.3, 192.9)
- moved C27 11.7 mm to (228.5, 204.6)
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Routing:
- net Net-(J501-Pad3): track 67.3 -> 0.00 mm, vias 1 -> 0
- net GND: track 1679.7 -> 1616.5 mm, vias 65 -> 67
- net A14_sel: track 61.6 -> 0.00 mm, vias 1 -> 0
- net Net-(U104-Pad4): track 61.0 -> 0.00 mm, vias 2 -> 0
- net Net-(U104-Pad9): track 60.5 -> 0.00 mm, vias 2 -> 0
- net Net-(U104-Pad7): track 55.5 -> 0.00 mm, vias 2 -> 0
- net A4: track 375.5 -> 328.6 mm
- net +5VA: track 2213.8 -> 2169.3 mm
- net Net-(D101-Pad1): track 42.5 -> 4.23 mm
- net D6XX: track 108.0 -> 74.2 mm, vias 5 -> 3
- net A6: track 320.3 -> 288.1 mm
- net A1: track 510.0 -> 477.9 mm
- net A7: track 303.7 -> 274.1 mm
- net A0: track 552.1 -> 523.6 mm
- net D1: track 569.8 -> 543.0 mm
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Other:
- board text removed: "74LVC2G74"

Commit message: Basic and os
Parts:
- moved C99 28.1 mm to (248.8, 181.9), turned to 180 degrees
- moved C203 25.3 mm to (247.3, 200.0), turned to 180 degrees
- moved U104 25.1 mm to (247.6, 188.5), turned to 0 degrees
- moved U105 25.0 mm to (246.8, 196.8), turned to 0 degrees
- moved C27 7.34 mm to (221.9, 201.4)
- moved U4 7.34 mm to (226.2, 189.8)
- moved U5 7.34 mm to (204.7, 189.8)
Routing:
- net D1: track 543.0 -> 602.6 mm, vias 11 -> 10
- net +5VA: track 2169.3 -> 2113.1 mm, vias 59 -> 55
- net D2: track 562.4 -> 617.3 mm, vias 11 -> 10
- net D0: track 549.3 -> 603.0 mm, vias 11 -> 10
- net A4: track 328.6 -> 366.4 mm
- net A9: track 290.5 -> 320.6 mm
- net OS: track 83.9 -> 57.0 mm
- net A6: track 288.1 -> 312.2 mm
- net A7: track 274.1 -> 297.0 mm
- net A1: track 477.9 -> 499.1 mm
- net A12: track 441.5 -> 460.6 mm
- net A8: track 297.3 -> 315.8 mm, vias 5 -> 3
- net GND: track 1616.5 -> 1598.1 mm
- net A0: track 523.6 -> 541.3 mm
- net A10: track 311.4 -> 327.0 mm, vias 6 -> 5
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
Commit message: Basic and OS
Parts:
- removed R75: 3k, Atari:R_Axial_DIN0207_L3.6mm_D2.2mm_P10.16mm_Horizontal
- removed W1: 0, Atari:R_Axial_DIN0207_L3.6mm_D2.2mm_P10.16mm_Horizontal
- U105: value 74LVC2G74 -> 74HC74; footprint Package_SO:TSSOP-8_3x3mm_P0.65mm -> Package_SO:SOIC-14_3.9x8.7mm_P1.27mm
- moved D100 61.7 mm to (200.9, 211.8), turned to 0 degrees
- moved R508 59.1 mm to (200.9, 209.4), turned to 0 degrees
- moved C99 59.1 mm to (200.8, 216.4), turned to 0 degrees
- moved D101 52.7 mm to (214.4, 209.9), turned to 0 degrees
- moved R509 50.1 mm to (214.4, 207.6), turned to 0 degrees
- moved C203 48.6 mm to (200.8, 214.1), turned to 0 degrees
- moved U104 47.7 mm to (208.1, 215.3)
- moved U105 36.6 mm to (215.6, 215.9)
- moved C207 17.1 mm to (233.9, 207.4)
- moved C209 17.1 mm to (243.4, 208.4)
- moved R502 17.1 mm to (231.5, 207.4)
- moved U100 17.1 mm to (231.3, 215.3)
- moved U101 17.1 mm to (240.8, 215.9)
- moved U102 17.1 mm to (250.4, 215.9)
- moved C208 17.1 mm to (262.4, 208.4)
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Connections:
- U105 pad 1: D6XX -> Net-(C203-Pad1)
- U105 pad 3: (no net) -> D6XX
- U105 pad 4: GND -> Net-(D101-Pad1)
- U105 pad 6: Net-(C203-Pad1) -> (no net)
- U105 pad 7: Net-(D101-Pad1) -> GND
- U105 pad 8: +5VA -> (no net)
- U22 pad 10: Net-(R75-Pad1) -> GND
Routing:
- net PB3: track 267.4 -> 346.0 mm, vias 3 -> 4
- net D6XX: track 74.2 -> 147.3 mm, vias 3 -> 5
- net PB2: track 265.3 -> 335.4 mm, vias 3 -> 4
- net GND: track 1598.1 -> 1664.7 mm, vias 67 -> 71
- net RST: track 544.4 -> 602.2 mm, vias 12 -> 13
- net +5VA: track 2113.1 -> 2163.9 mm, vias 55 -> 50
- net Net-(U104-Pad7): track 0.00 -> 44.1 mm, vias 0 -> 1
- net RD5: track 340.5 -> 297.0 mm
- net Net-(C203-Pad1): track 0.00 -> 32.3 mm, vias 0 -> 2
- net Net-(U104-Pad9): track 0.00 -> 32.0 mm
- net Net-(U104-Pad4): track 0.00 -> 27.8 mm, vias 0 -> 1
- net CCTL: track 246.6 -> 220.7 mm
- net S5: track 265.1 -> 244.6 mm, vias 6 -> 4
- net A16_sel: track 18.9 -> 0.00 mm, vias 1 -> 0
- net A15_sel: track 16.0 -> 0.00 mm, vias 1 -> 0
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Other:
- board text removed: "A14"
- board text removed: "A15"
- board text removed: "A16"
- board text removed: "Basic on/off"
- board text removed: "OS on/off"
- board text removed: "TTP"
