File: Atari 130XE 1MB smd.kicad_pcb (KiCad board)
At the start: 2 copper layers, 324 x 204 mm, 369 parts, among them J1 SIO, J10 Mem_on_off, J2 Video, J201 Diagnostic, J202 Diag, J210 Diag, J24 Cartridge, J4 Expansion, J5 Joystick_Port, J50 Test_signal, J500 Basic_sel, J501 TPP_sel, J51 To_GND, J6 Joystick_Port, J7 Power, J8 Keyboard, Q1 2N3904, Q10 PN2222A, Q101 BC849, Q11 PN2222A, Q2 2N3904, Q3 2N3904, Q4 2N3906, Q6 2N3904, SW1 Switch_power_on, U10 DRAM_4464, U100 74LS157, U101 74LS74, U102 74HC02, U103 74HC02, U104 74LS157, U105 74HC74, U17 GTIA, U18 74LS08, U19 LM555, U2 74LS138, U20 4050, U21 74LS74, U22 POKEY, U23 PIA, U24 CD4051B, U25 CD4051B, U3 MMU, U4 27C010, U40 GAL20V8_DIP, U41 74LS157, U42 74LS175, U43 DRAM_1MB_4bit, U44 DRAM_1MB_4bit, U45 74HC04, U5 27C010, U6 Freddie, U7 Antic, U8 Sally, U9 DRAM_4464, Y1 Crystal, Y2 4,43 MHz

Commit message: text on top
Other:
- board text added: "74HCT04"
Changed lines of the file:
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@@
   (general
     (thickness 1.6)
-    (drawings 93)
+    (drawings 94)
     (tracks 7954)
     (zones 0)
@@
   )
   (setup
-    (last_trace_width 0.6096)
+    (last_trace_width 0.25)
     (user_trace_width 0.254)
     (user_trace_width 0.3048)
@@
     (tags "SOIC 1.27")
     (attr smd)
-    (fp_text reference U45 (at 0 -5.375 90) (layer F.SilkS)
+    (fp_text reference U45 (at -0.127 -0.3556 180) (layer F.SilkS)
       (effects (font (size 1 1) (thickness 0.15)))
     )
@@
       (net 1 GND))
   )
+  (gr_text 74HCT04 (at 78.867 173.3296 90) (layer F.SilkS)
+    (effects (font (size 1 1) (thickness 0.15)))
+  )
   (gr_text "RAS 1" (at 88.1634 186.3344 90) (layer F.SilkS)
     (effects (font (size 1 1) (thickness 0.15)))
@@
   (segment (start 74.0918 155.448) (end 74.0918 180.0352) (width 0.4064) (layer F.Cu) (net 20))
   (segment (start 74.3585 155.1813) (end 74.0918 155.448) (width 0.4064) (layer F.Cu) (net 20))
-  (via (at 68.0212 151.3078) (size 0.9) (drill 0.5) (layers F.Cu B.Cu) (net 322))
-  (segment (start 68.0085 153.289) (end 68.0085 151.3205) (width 0.4064) (layer F.Cu) (net 322))
-  (segment (start 68.0085 151.3205) (end 68.0212 151.3078) (width 0.4064) (layer F.Cu) (net 322))
-  (via (at 68.0212 136.8806) (size 0.9) (drill 0.5) (layers F.Cu B.Cu) (net 322))
-  (segment (start 68.0212 151.3078) (end 68.0212 136.8806) (width 0.4064) (layer B.Cu) (net 322))
-  (segment (start 68.0212 138.9253) (end 68.0085 138.938) (width 0.4064) (layer F.Cu) (net 322))
-  (segment (start 68.0212 136.8806) (end 68.0212 138.9253) (width 0.4064) (layer F.Cu) (net 322))
-  (segment (start 74.5484 113.5882) (end 74.5484 111.4952) (width 0.4064) (layer F.Cu) (net 322))
-  (segment (start 75.819 114.8588) (end 74.5484 113.5882) (width 0.4064) (layer F.Cu) (net 322))
-  (segment (start 75.819 119.507) (end 75.819 114.8588) (width 0.4064) (layer F.Cu) (net 322))
-  (segment (start 74.5484 124.1752) (end 74.5484 120.7776) (width 0.4064) (layer F.Cu) (net 322))
-  (segment (start 74.5484 120.7776) (end 75.819 119.507) (width 0.4064) (layer F.Cu) (net 322))
   (via (at 87.249 200.5584) (size 0.9) (drill 0.5) (layers F.Cu B.Cu) (net 21))
-  (segment (start 68.0085 157.2387) (end 68.0085 153.289) (width 0.4064) (layer F.Cu) (net 322))
-  (via (at 68.0085 159.9819) (size 0.9) (drill 0.5) (layers F.Cu B.Cu) (net 322))
-  (segment (start 68.0085 159.9819) (end 68.0085 157.2387) (width 0.4064) (layer F.Cu) (net 322))
-  (segment (start 74.5484 126.1878) (end 74.5484 124.1752) (width 0.4064) (layer F.Cu) (net 322))
-  (segment (start 68.0212 136.8806) (end 68.0212 136.244204) (width 0.4064) (layer F.Cu) (net 322))
-  (segment (start 68.527804 135.7376) (end 70.38203 135.7376) (width 0.4064) (layer F.Cu) (net 322))
-  (segment (start 70.38203 135.7376) (end 72.771 133.34863) (width 0.4064) (layer F.Cu) (net 322))
-  (segment (start 72.771 133.34863) (end 72.771 127.9652) (width 0.4064) (layer F.Cu) (net 322))
-  (segment (start 68.0212 136.244204) (end 68.527804 135.7376) (width 0.4064) (layer F.Cu) (net 322))
-  (segment (start 72.771 127.9652) (end 74.5484 126.1878) (width 0.4064) (layer F.Cu) (net 322))
   (via (at 68.2371 177.8889) (size 0.8) (drill 0.4) (layers F.Cu B.Cu) (net 21))
   (segment (start 65.9384 180.1876) (end 68.2371 177.8889) (width 0.254) (layer B.Cu) (net 21))
@@
   (segment (start 87.249 174.2636) (end 86.8484 173.863) (width 0.4064) (layer F.Cu) (net 320))
   (segment (start 85.979 170.02) (end 87.249 170.02) (width 0.4064) (layer F.Cu) (net 321))
+  (via (at 68.0212 151.3078) (size 0.9) (drill 0.5) (layers F.Cu B.Cu) (net 322))
+  (segment (start 68.0085 153.289) (end 68.0085 151.3205) (width 0.4064) (layer F.Cu) (net 322))
+  (segment (start 68.0085 151.3205) (end 68.0212 151.3078) (width 0.4064) (layer F.Cu) (net 322))
+  (via (at 68.0212 136.8806) (size 0.9) (drill 0.5) (layers F.Cu B.Cu) (net 322))
+  (segment (start 68.0212 151.3078) (end 68.0212 136.8806) (width 0.4064) (layer B.Cu) (net 322))
+  (segment (start 68.0212 138.9253) (end 68.0085 138.938) (width 0.4064) (layer F.Cu) (net 322))
+  (segment (start 68.0212 136.8806) (end 68.0212 138.9253) (width 0.4064) (layer F.Cu) (net 322))
+  (segment (start 74.5484 113.5882) (end 74.5484 111.4952) (width 0.4064) (layer F.Cu) (net 322))
+  (segment (start 75.819 114.8588) (end 74.5484 113.5882) (width 0.4064) (layer F.Cu) (net 322))
+  (segment (start 75.819 119.507) (end 75.819 114.8588) (width 0.4064) (layer F.Cu) (net 322))
+  (segment (start 74.5484 124.1752) (end 74.5484 120.7776) (width 0.4064) (layer F.Cu) (net 322))
+  (segment (start 74.5484 120.7776) (end 75.819 119.507) (width 0.4064) (layer F.Cu) (net 322))
+  (segment (start 68.0085 157.2387) (end 68.0085 153.289) (width 0.4064) (layer F.Cu) (net 322))
+  (via (at 68.0085 159.9819) (size 0.9) (drill 0.5) (layers F.Cu B.Cu) (net 322))
+  (segment (start 68.0085 159.9819) (end 68.0085 157.2387) (width 0.4064) (layer F.Cu) (net 322))
+  (segment (start 74.5484 126.1878) (end 74.5484 124.1752) (width 0.4064) (layer F.Cu) (net 322))
+  (segment (start 68.0212 136.8806) (end 68.0212 136.244204) (width 0.4064) (layer F.Cu) (net 322))
+  (segment (start 68.527804 135.7376) (end 70.38203 135.7376) (width 0.4064) (layer F.Cu) (net 322))
+  (segment (start 70.38203 135.7376) (end 72.771 133.34863) (width 0.4064) (layer F.Cu) (net 322))
+  (segment (start 72.771 133.34863) (end 72.771 127.9652) (width 0.4064) (layer F.Cu) (net 322))
+  (segment (start 68.0212 136.244204) (end 68.527804 135.7376) (width 0.4064) (layer F.Cu) (net 322))
+  (segment (start 72.771 127.9652) (end 74.5484 126.1878) (width 0.4064) (layer F.Cu) (net 322))
   (segment (start 80.645 179.2882) (end 83.1342 179.2882) (width 0.4064) (layer F.Cu) (net 322))
   (segment (start 83.1342 179.2882) (end 85.6234 179.2882) (width 0.4064) (layer F.Cu) (net 322))

Commit message: Gerber
Parts:
- removed JP1, JP2, JP3, JP4: SolderJumper_2_Open, Jumper:SolderJumper-2_P1.3mm_Open_RoundedPad1.0x1.5mm
- added J12: Conn_02x04_Odd_Even, Connector_PinHeader_2.00mm:PinHeader_2x04_P2.00mm_Vertical, F.Cu at (81.4, 181.4)
Connections:
- U20 pad 16: +5VA -> (no net)
Routing:
- net RAS: track 66.5 -> 68.0 mm
- net Net-(J12-Pad6): track 9.62 -> 10.9 mm, vias 2 -> 1
- net Net-(J12-Pad4): track 14.5 -> 15.5 mm, vias 2 -> 1
- net Net-(J12-Pad8): track 4.89 -> 5.81 mm
- net RAS_out: track 128.2 -> 127.6 mm, vias 6 -> 5
- net GND: vias 164 -> 167

Commit message: SIO2SD schema
Parts:
- removed J201: Diagnostic, Connector_PinHeader_2.54mm:PinHeader_1x04_P2.54mm_Vertical
- added 74AC245: 74HC245, Package_SO:SOIC-20W_7.5x12.8mm_P1.27mm, F.Cu at (312.7, 88.3)
- added ATMEGA32: ATmega32-16AU, Package_QFP:TQFP-44_10x10mm_P0.8mm, F.Cu at (297.0, 88.2)
- added C220: 22p, Capacitor_SMD:C_1206_3216Metric_Pad1.42x1.75mm_HandSolder, F.Cu at (294.9, 97.0)
- added C221: 22p, Capacitor_SMD:C_1206_3216Metric_Pad1.42x1.75mm_HandSolder, F.Cu at (300.0, 97.0)
- added C222: 100n, Capacitor_SMD:C_1206_3216Metric_Pad1.42x1.75mm_HandSolder, F.Cu at (305.3, 101.8)
- added C223: 100n, Capacitor_SMD:C_1206_3216Metric_Pad1.42x1.75mm_HandSolder, F.Cu at (316.2, 80.1)
- added C224: 100n, Capacitor_SMD:C_1206_3216Metric_Pad1.42x1.75mm_HandSolder, F.Cu at (288.4, 88.1)
- added D200: 1N4001, Diode_SMD:D_MELF, F.Cu at (316.6, 111.6)
- added J204: ISP, Connector_IDC:IDC-Header_2x03_P2.54mm_Vertical, F.Cu at (326.0, 111.6)
- added LED: SIOLED, Connector_PinHeader_2.54mm:PinHeader_1x02_P2.54mm_Vertical, F.Cu at (320.8, 98.9)
- added MICRO SD: Micro_SD_Card, Jacek:MCC SDMicro, F.Cu at (330.8, 85.8)
- added R220: 10k, Resistor_SMD:R_1206_3216Metric_Pad1.42x1.75mm_HandSolder, F.Cu at (304.0, 110.7)
- added R221: 4k7, Resistor_SMD:R_1206_3216Metric_Pad1.42x1.75mm_HandSolder, F.Cu at (306.4, 110.7)
- added R222: 470, Resistor_SMD:R_1206_3216Metric_Pad1.42x1.75mm_HandSolder, F.Cu at (317.6, 99.5)
- added SIO: SIO, Connector_PinHeader_2.00mm:PinHeader_2x03_P2.00mm_Vertical, F.Cu at (313.2, 109.7)
- added U202: LM2936-3.3, Package_TO_SOT_SMD:SOT-223-3_TabPin2, F.Cu at (310.9, 100.7)
- added Y200: Crystal, Crystal:Crystal_HC18-U_Vertical, F.Cu at (299.8, 101.1)
- moved L19 49.9 mm to (322.6, 141.0), turned to 180 degrees
- moved L26 48.6 mm to (335.3, 133.7), turned to 180 degrees
- moved L20 41.9 mm to (322.6, 136.4), turned to 180 degrees
- moved L27 41.0 mm to (335.3, 129.1), turned to 180 degrees
- moved FB12 38.5 mm to (346.2, 179.3), turned to 0 degrees
- moved L25 38.4 mm to (346.2, 175.3), turned to 180 degrees
- moved FB102 38.4 mm to (346.2, 171.2), turned to 0 degrees
- moved C102 38.3 mm to (345.5, 168.0), turned to 0 degrees
- moved L21 34.2 mm to (322.6, 131.8), turned to 180 degrees
- moved L28 33.8 mm to (335.3, 124.4), turned to 180 degrees
- moved L30 28.5 mm to (330.2, 150.9)
- moved C97 28.5 mm to (329.6, 141.5)
- moved C96 28.5 mm to (329.6, 143.8)
- moved L23 28.5 mm to (330.3, 147.0)
- moved L29 27.7 mm to (335.3, 119.8), turned to 180 degrees
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Routing:
- net GND: track 1822.3 -> 1708.6 mm, vias 167 -> 169
- net +5VA: track 2465.8 -> 2420.9 mm, vias 59 -> 58
- net DATA_OUT: track 100.8 -> 145.1 mm
- net DATA_IN: track 94.6 -> 136.4 mm
- net CLK_OUT: track 92.0 -> 131.6 mm
- net CLK_IN: track 83.8 -> 122.8 mm
- net Net-(R19-Pad1): track 29.8 -> 68.2 mm
- net TRIG0: track 36.6 -> 74.2 mm
- net POT_A1: track 91.4 -> 125.6 mm
- net POT_B0: track 66.5 -> 100.3 mm, vias 3 -> 1
- net Net-(C102-Pad1): track 93.3 -> 126.8 mm, vias 2 -> 1
- net TRIG1: track 70.1 -> 103.5 mm, vias 3 -> 1
- net POT_A0: track 61.8 -> 94.1 mm, vias 3 -> 1
- net Net-(R86-Pad2): track 56.4 -> 88.2 mm
- net POT_B1: track 95.9 -> 127.2 mm
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Other:
- board text removed: "Clk_out"
- board text removed: "Data_in"
- board text removed: "Data_out"

Commit message: Final Atmega32
Parts:
- added C225: 22n, Capacitor_SMD:C_1206_3216Metric_Pad1.42x1.75mm_HandSolder, F.Cu at (320.6, 81.2)
- added C226: 22n, Capacitor_SMD:C_1206_3216Metric_Pad1.42x1.75mm_HandSolder, F.Cu at (318.1, 81.2)
- added C227: 22n, Capacitor_SMD:C_1206_3216Metric_Pad1.42x1.75mm_HandSolder, F.Cu at (315.5, 81.2)
- added C228: 22n, Capacitor_SMD:C_1206_3216Metric_Pad1.42x1.75mm_HandSolder, F.Cu at (313.0, 81.2)
- added C229: 22n, Capacitor_SMD:C_1206_3216Metric_Pad1.42x1.75mm_HandSolder, F.Cu at (310.5, 81.2)
- added C230: 10n, Capacitor_SMD:C_1206_3216Metric_Pad1.42x1.75mm_HandSolder, F.Cu at (337.9, 83.4)
- added C231: 220uF, Capacitor_Tantalum_SMD:CP_EIA-7343-40_Kemet-Y_Pad2.25x2.55mm_HandSolder, F.Cu at (340.0, 87.4)
- added J207: LCD 2x16, Connector_PinHeader_2.54mm:PinHeader_1x08_P2.54mm_Vertical, F.Cu at (288.8, 76.8)
- added J208: SD buttons, Connector_PinHeader_2.54mm:PinHeader_1x05_P2.54mm_Vertical, F.Cu at (310.5, 76.8)
- added J209: SD config, Connector_PinHeader_2.54mm:PinHeader_2x03_P2.54mm_Vertical, F.Cu at (106.2, 75.0)
- added J211: SIOLED2, Connector_PinHeader_2.54mm:PinHeader_1x02_P2.54mm_Vertical, F.Cu at (318.9, 104.9)
- added J212: SIOLED3, Connector_PinHeader_2.54mm:PinHeader_1x02_P2.54mm_Vertical, F.Cu at (315.3, 104.9)
- added R223: 220, Resistor_SMD:R_1206_3216Metric_Pad1.42x1.75mm_HandSolder, F.Cu at (340.1, 103.2)
- added R224: 220, Resistor_SMD:R_1206_3216Metric_Pad1.42x1.75mm_HandSolder, F.Cu at (340.1, 105.5)
- J203: renamed from MICRO SD
- J206: renamed from LED; value SIOLED -> SIOLED1
- R222: value 470 -> 220
- moved R222 22.5 mm to (340.1, 101.0), turned to 180 degrees
- moved C223 21.4 mm to (306.3, 99.1)
- moved J203 20.4 mm to (347.4, 74.1), turned to 270 degrees
- moved J206 6.27 mm to (322.5, 104.9), turned to 180 degrees
- moved C222 4.62 mm to (302.8, 105.7)
- moved U202 4.62 mm to (308.5, 104.6)
- moved U201 4.25 mm to (309.5, 91.1)
- moved Q4 3.36 mm to (258.3, 87.0)
- moved C224 2.34 mm to (286.3, 88.9)
- moved C220 2.13 mm to (292.7, 97.0)
- moved U200 2.13 mm to (294.9, 88.2)
- moved Y200 2.13 mm to (297.7, 101.1)
- moved C221 2.13 mm to (297.9, 97.0)
- moved J205 1.84 mm to (313.1, 111.5)
- moved R220 1.84 mm to (303.9, 112.6)
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- renumbered SIO to J205, ATMEGA32 to U200, 74AC245 to U201
Connections:
- U200 pad 14: (no net) -> Net-(J209-Pad1)
- U200 pad 15: (no net) -> Net-(J209-Pad3)
- U200 pad 16: (no net) -> Net-(J209-Pad5)
- U200 pad 24: (no net) -> Net-(J212-Pad2)
- U200 pad 25: (no net) -> Net-(J211-Pad2)
- U200 pad 30: (no net) -> Net-(J207-Pad8)
- U200 pad 31: (no net) -> Net-(J207-Pad7)
- U200 pad 32: (no net) -> Net-(J207-Pad6)
- U200 pad 33: (no net) -> Net-(J207-Pad5)
- U200 pad 34: (no net) -> Net-(J207-Pad4)
- U200 pad 35: (no net) -> Net-(J207-Pad3)
- U200 pad 36: (no net) -> Net-(J207-Pad2)
- U200 pad 37: (no net) -> Net-(J207-Pad1)
- U200 pad 40: (no net) -> Net-(C225-Pad2)
- U200 pad 41: (no net) -> Net-(C226-Pad2)
- U200 pad 42: (no net) -> Net-(C227-Pad2)
- U200 pad 43: (no net) -> Net-(C228-Pad2)
- U200 pad 44: (no net) -> Net-(C229-Pad2)
Routing:
- net Net-(J209-Pad5): track 0.00 -> 222.9 mm, vias 0 -> 5
- net Net-(J209-Pad3): track 0.00 -> 221.1 mm, vias 0 -> 5
- net Net-(J209-Pad1): track 0.00 -> 221.0 mm, vias 0 -> 5
- net A16_sel: track 584.4 -> 480.7 mm
- net +5VA: track 2420.9 -> 2524.3 mm, vias 58 -> 62
- net +3V3: track 0.00 -> 102.6 mm, vias 0 -> 4
- net Net-(J204-Pad5): track 0.00 -> 69.4 mm, vias 0 -> 3
- net Net-(J204-Pad4): track 0.00 -> 68.1 mm, vias 0 -> 1
- net Net-(J203-Pad9): track 0.00 -> 64.7 mm, vias 0 -> 2
- net Net-(J203-Pad7): track 0.00 -> 63.4 mm
- net Net-(J204-Pad3): track 0.00 -> 62.0 mm, vias 0 -> 1
- net Net-(J204-Pad1): track 0.00 -> 59.6 mm, vias 0 -> 1
- net Net-(J203-Pad5): track 0.00 -> 47.2 mm
- net Net-(C226-Pad2): track 0.00 -> 46.3 mm, vias 0 -> 1
- net RST: track 612.4 -> 658.6 mm, vias 12 -> 13
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Other:
- board text added: "A14, A15, A16 Bank sel"
- board text added: "ATMEGA32"
- board text added: "BASIC A14"
- board text added: "BASIC A15"
- board text added: "BASIC A16"
- board text added: "BASIC Sel"
- board text added: "OFF - Carts"
- board text added: "OFF - TTP"
- board text added: "ON - ATARI OS"
- board text added: "ON - BASIC"
- board text added: "PD5"
- board text added: "PD6"
- board text added: "PD7"
- board text added: "SIO2SD pins"
- board text added: "TTP Rst"
- board text added: "TTP Sel"

Commit message: final inspection
Parts:
- added J213: SD_conn, Connector_PinHeader_2.54mm:PinHeader_1x07_P2.54mm_Vertical, F.Cu at (332.5, 68.5)
Routing:
- net +5VA: track 2524.3 -> 2532.0 mm, vias 62 -> 60
- net AUDIO: track 101.4 -> 107.2 mm
- net Net-(J203-Pad7): track 63.4 -> 68.2 mm
- net +3V3: track 102.6 -> 106.5 mm
- net Net-(J203-Pad5): track 47.2 -> 50.5 mm
- net MONO: track 31.1 -> 33.5 mm
- net Net-(J203-Pad9): track 64.7 -> 66.6 mm
- net D7: track 446.8 -> 448.5 mm
- net Net-(J203-Pad3): track 46.2 -> 47.4 mm
- net Net-(J203-Pad2): track 45.8 -> 47.0 mm
- net GND: track 1679.5 -> 1680.0 mm, vias 209 -> 240
Other:
- board text added: "3,3V"
- board text added: "74LS02"
- board text added: "COM"
- board text added: "CS"
- board text added: "MISO"
- board text added: "MOSI"
- board text added: "SCK"
- board text added: "SD conn"
- board text removed: "Clk_in"
