File: Atari 130XE 1MB smd.kicad_pcb (KiCad board)
At the start: 2 copper layers, 324 x 204 mm, 397 parts, among them J1 SIO, J10 Mem_on_off, J12 Conn_02x04_Odd_Even, J2 Video, J202 Diag, J203 Micro_SD_Card, J204 ISP, J205 SIO, J206 SIOLED1, J207 LCD 2x16, J208 SD buttons, J209 SD config, J210 Diag, J211 SIOLED2, J212 SIOLED3, J213 SD_conn, J24 Cartridge, J4 Expansion, J5 Joystick_Port, J50 Test_signal, J500 Basic_sel, J501 TPP_sel, J51 To_GND, J6 Joystick_Port, J7 Power, J8 Keyboard, Q1 2N3904, Q10 PN2222A, Q101 BC849, Q11 PN2222A, Q2 2N3904, Q3 2N3904, Q4 2N3906, Q6 2N3904, SW1 Switch_power_on, U10 DRAM_4464, U100 74LS157, U101 74LS74, U102 74HC02, U103 74HC02, U104 74LS157, U105 74HC74, U17 GTIA, U18 74LS08, U19 LM555, U2 74LS138, U20 4050, U200 ATmega32-16AU, U201 74HC245, U202 LM2936-3.3, U21 74LS74, U22 POKEY, U23 PIA, U24 CD4051B, U25 CD4051B, U3 MMU, U4 27C010, U40 GAL20V8_DIP, U41 74LS157, U42 74LS175, U43 DRAM_1MB_4bit, U44 DRAM_1MB_4bit, U45 74HC04, U5 27C010, U6 Freddie, U7 Antic, U8 Sally, U9 DRAM_4464, Y1 Crystal, Y2 4,43 MHz, Y200 Crystal

Commit message: Final inspection
Parts:
- C36, C37: footprint Capacitor_THT:C_Axial_L3.8mm_D2.6mm_P7.50mm_Horizontal -> Capacitor_SMD:C_1206_3216Metric_Pad1.42x1.75mm_HandSolder
- Y200: value Crystal -> 14,31818 MHz
- moved C36 1.50 mm to (87.8, 125.7), turned to 270 degrees
- moved C37 1.50 mm to (87.8, 110.0)
- moved J1 1.00 mm to (328.9, 61.9)
Routing:
- net GND: track 1680.0 -> 1657.2 mm, vias 240 -> 236
- net +5VA: track 2532.0 -> 2535.8 mm
- net RA0: track 114.9 -> 117.1 mm
- net Net-(R127-Pad2): track 62.0 -> 59.9 mm
- net MTR_CLR: track 72.1 -> 70.2 mm
- net Net-(R126-Pad2): track 60.3 -> 58.6 mm
- net Net-(R125-Pad2): track 59.2 -> 58.0 mm
- net SIOAUDIO: track 253.5 -> 252.4 mm
- net PB6: track 303.1 -> 304.1 mm
- net PB0: track 281.1 -> 282.1 mm
- net PB4: track 261.5 -> 262.4 mm
- net PB3: track 331.9 -> 332.9 mm
- net RAS: track 68.0 -> 67.0 mm
- net PB1: track 293.2 -> 294.2 mm
- net PB2: track 333.5 -> 334.4 mm
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Other:
- board text added: "14,31818 MHz"

Commit message: Gerber
Other:
- board text added: "14,18757 MHz"
- board text removed: "74HC02"
Changed lines of the file:
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@@
   (general
     (thickness 1.6)
-    (drawings 120)
+    (drawings 117)
     (tracks 8573)
     (zones 0)
@@
   )
   (setup
-    (last_trace_width 1.524)
+    (last_trace_width 0.25)
     (user_trace_width 0.254)
     (user_trace_width 0.3048)
@@
     (descr "Through hole straight pin header, 1x05, 2.54mm pitch, single row")
     (tags "Through hole pin header THT 1x05 2.54mm single row")
-    (fp_text reference J208 (at -2.2352 13.462 180) (layer F.SilkS)
+    (fp_text reference J208 (at 0.127 13.589 180) (layer F.SilkS)
       (effects (font (size 1 1) (thickness 0.15)))
     )
@@
     (descr "Through hole straight pin header, 1x08, 2.54mm pitch, single row")
     (tags "Through hole pin header THT 1x08 2.54mm single row")
-    (fp_text reference J207 (at 0 -2.33 90) (layer F.SilkS)
+    (fp_text reference J207 (at 0.6604 -3.683 180) (layer F.SilkS)
       (effects (font (size 1 1) (thickness 0.15)))
     )
@@
   (module "Jacek:MCC SDMicro" (layer F.Cu)
     (at 347.4466 74.0918 270)
-    (fp_text reference J203 (at 0.4572 -7.493 90) (layer F.SilkS)
+    (fp_text reference J203 (at -0.4572 7.7724 270) (layer F.SilkS)
       (effects (font (size 1 1) (thickness 0.15)))
     )
@@
     (descr "Through hole straight pin header, 2x04, 2.00mm pitch, double rows")
     (tags "Through hole pin header THT 2x04 2.00mm double row")
-    (fp_text reference J12 (at 1 -2.06 90) (layer F.SilkS)
+    (fp_text reference J12 (at 1.143 -3.1496 180) (layer F.SilkS)
       (effects (font (size 1 1) (thickness 0.15)))
     )
@@
     (descr "Through hole straight pin header, 1x02, 2.54mm pitch, single row")
     (tags "Through hole pin header THT 1x02 2.54mm single row")
-    (fp_text reference J51 (at 0 -2.33 90) (layer F.SilkS)
+    (fp_text reference J51 (at 0.1016 -2.8702 180) (layer F.SilkS)
       (effects (font (size 1 1) (thickness 0.15)))
     )
@@
     (descr "Through hole straight pin header, 2x05, 2.54mm pitch, double rows")
     (tags "Through hole pin header THT 2x05 2.54mm double row")
-    (fp_text reference J50 (at 1.27 -2.6924) (layer F.SilkS)
+    (fp_text reference J50 (at 1.3208 12.6238) (layer F.SilkS)
       (effects (font (size 1 1) (thickness 0.15)))
     )
@@
     (tags "resistor handsolder")
     (attr smd)
-    (fp_text reference R128 (at -3.5814 0.4572 270) (layer F.SilkS)
+    (fp_text reference R128 (at -3.556 0.2032 270) (layer F.SilkS)
       (effects (font (size 1 1) (thickness 0.15)))
     )
@@
     (tags "resistor handsolder")
     (attr smd)
-    (fp_text reference R83 (at 0 -1.82) (layer F.SilkS)
+    (fp_text reference R83 (at -4.1656 0.1016) (layer F.SilkS)
       (effects (font (size 1 1) (thickness 0.15)))
     )
@@
     (tags "capacitor handsolder")
     (attr smd)
-    (fp_text reference C76 (at 4.0894 -0.0762 180) (layer F.SilkS)
+    (fp_text reference C76 (at 4.1148 -0.0762 180) (layer F.SilkS)
       (effects (font (size 1 1) (thickness 0.15)))
     )
@@
     (tags "capacitor handsolder")
     (attr smd)
-    (fp_text reference C75 (at -3.81 -0.0254 180) (layer F.SilkS)
+    (fp_text reference C75 (at 4.1402 -0.1524 180) (layer F.SilkS)
       (effects (font (size 1 1) (thickness 0.15)))
     )
@@
     (tags "capacitor handsolder")
     (attr smd)
-    (fp_text reference C124 (at 4.80314 0.0508 270) (layer F.SilkS)
+    (fp_text reference C124 (at -0.0127 2.159 270) (layer F.SilkS)
       (effects (font (size 1 1) (thickness 0.15)))
     )
@@
   (module Atari:Joystick_Pport (layer F.Cu)
     (at 359.8884 77.8752 270)
-    (fp_text reference J6 (at 22.4294 9.9526 270) (layer F.SilkS)
+    (fp_text reference J6 (at 13.0568 12.899 270) (layer F.SilkS)
       (effects (font (size 1 1) (thickness 0.15)))
     )
@@
   (module Atari:Joystick_Pport (layer F.Cu)
     (at 359.8884 45.8752 270)
-    (fp_text reference J5 (at 22.1714 10.0034 270) (layer F.SilkS)
+    (fp_text reference J5 (at 12.2908 12.772 270) (layer F.SilkS)
       (effects (font (size 1 1) (thickness 0.15)))
     )
@@
     (descr "Crystal THT HC-18/U, http://5hertz.com/pdfs/04404_D.pdf")
     (tags "THT crystalHC-18/U")
-    (fp_text reference Y1 (at 2.286 -0.1524) (layer F.SilkS)
+    (fp_text reference Y1 (at 2.2606 -3.43154) (layer F.SilkS)
       (effects (font (size 1 1) (thickness 0.15)))
     )
@@
       (net 1 GND))
   )
+  (gr_text "14,18757 MHz" (at 83.7692 229.616) (layer F.SilkS)
+    (effects (font (size 1 1) (thickness 0.1)))
+  )
   (gr_text "14,31818 MHz" (at 293.8018 104.648) (layer F.SilkS)
     (effects (font (size 1 1) (thickness 0.15)))
@@
     (effects (font (size 1 1) (thickness 0.15)))
   )
-  (gr_text 74HCT04 (at 78.867 173.3296 90) (layer F.SilkS)
+  (gr_text 74HCT04 (at 81.8134 168.021) (layer F.SilkS)
     (effects (font (size 1 1) (thickness 0.15)))
   )
@@
     (effects (font (size 1 1) (thickness 0.15)))
   )
-  (gr_text Diagnostic (at 65.786 178.6382) (layer F.SilkS)
+  (gr_text Diagnostic (at 66.1416 180.3908) (layer F.SilkS)
     (effects (font (size 1 1) (thickness 0.15)))
   )
@@
     (effects (font (size 1 1) (thickness 0.15)))
   )
-  (gr_text 74LS157 (at 101.2444 163.7792 90) (layer F.SilkS)
-    (effects (font (size 1 1) (thickness 0.15)))
-  )
-  (gr_text 74LS175 (at 101.1936 154.1018 90) (layer F.SilkS)
-    (effects (font (size 1 1) (thickness 0.15)))
-  )
-  (gr_text 74HC02 (at 270.4084 236.1184) (layer F.SilkS)
-    (effects (font (size 1 1) (thickness 0.15)))
-  )
-  (gr_text 74HC02 (at 261.493 236.1184) (layer F.SilkS)
-    (effects (font (size 1 1) (thickness 0.15)))
-  )
-  (gr_text 74LS74 (at 251.8156 236.1184) (layer F.SilkS)
+  (gr_text 74LS157 (at 103.4796 162.6108) (layer F.SilkS)
     (effects (font (size 1 1) (thickness 0.15)))
   )
-  (gr_text 74LS157 (at 242.1636 236.1184) (layer F.SilkS)
+  (gr_text 74LS175 (at 103.5304 152.9842) (layer F.SilkS)
     (effects (font (size 1 1) (thickness 0.15)))
   )
-  (gr_text 1MB/512kB (at 98.171 170.7642 90) (layer F.SilkS)
+  (gr_text 1MB/512kB (at 97.9424 172.7454 90) (layer F.SilkS)
     (effects (font (size 0.8 0.8) (thickness 0.12)))
   )
-  (gr_text on/off (at 90.805 171.0944 90) (layer F.SilkS)
+  (gr_text on/off (at 90.805 173.101 90) (layer F.SilkS)
     (effects (font (size 1 1) (thickness 0.15)))
   )
@@
     (effects (font (size 1.1 1.1) (thickness 0.16)))
   )
-  (gr_text Composite (at 148.6916 62.3062) (layer F.SilkS)
+  (gr_text Composite (at 150.1394 61.976) (layer F.SilkS)
     (effects (font (size 1.1 1.1) (thickness 0.16)))
   )
