File: Atari 130XE 1MB smd.sch (KiCad schematic (older format))
At the start: 0 parts

Commit message: SIO2SD schema
Changed lines of the file:
@@
 $Descr A4 11693 8268
 encoding utf-8
-Sheet 1 16
+Sheet 1 17
 Title ""
 Date ""
@@
 F1 "Simm_Expansion.sch" 50
 $EndSheet
+$Sheet
+S 5850 4475 1225 1175
+U 62DF8815
+F0 "SIO2SD" 50
+F1 "SIO2SD.sch" 50
+$EndSheet
 $EndSCHEMATC
