File: BASIC.sch (KiCad schematic (older format))
At the start: 19 parts, among them J500 Basic_sel, U100 74LS157, U101 74LS74, U102 74HC02, U103 74HC02, U4 27C010

Commit message: SMD continue
Connections:
- net A14_sel: now also J500.3 (Pin_3); no longer J500.5 (Pin_5)
- net A15_sel: now also J500.5 (Pin_5); no longer J500.3 (Pin_3)
- net A16_sel: now also J500.7 (Pin_7); no longer J500.1 (Pin_1)
- net at R506.2, U100.1 (S): now also J500.1 (Pin_1); no longer J500.7 (Pin_7)
Changed lines of the file:
@@
 	1    0    0    -1
 $EndComp
-Wire Wire Line
-	10250 1650 9800 1650
-Wire Wire Line
-	10250 1750 9525 1750
-Wire Wire Line
-	10250 1850 9250 1850
 $Comp
 L power:+5VA #PWR0275
@@
 Connection ~ 9250 1275
 Wire Wire Line
-	9250 1275 9250 1850
+	9250 1275 9250 1750
 Wire Wire Line
 	8675 1400 9525 1400
 Connection ~ 9525 1400
 Wire Wire Line
-	9525 1400 9525 1750
-Wire Wire Line
 	8675 1525 9800 1525
 Connection ~ 9800 1525
 Wire Wire Line
-	9800 1525 9800 1650
-Wire Wire Line
 	6875 4400 6875 1950
 Wire Wire Line
@@
 Wire Wire Line
 	8975 1150 8975 1950
-Connection ~ 8975 1950
-Wire Wire Line
-	8975 1950 10250 1950
 Text GLabel 800  6350 0    50   Input ~ 0
 RD5
@@
 	7025 3600 7300 3600
 Connection ~ 7300 4500
+Wire Wire Line
+	9800 1950 10250 1950
+Wire Wire Line
+	9800 1525 9800 1950
+Wire Wire Line
+	8975 1950 9700 1950
+Wire Wire Line
+	9700 1950 9700 1650
+Wire Wire Line
+	9700 1650 10250 1650
+Connection ~ 8975 1950
+Wire Wire Line
+	9525 1850 10250 1850
+Wire Wire Line
+	9525 1400 9525 1850
+Wire Wire Line
+	10250 1750 9250 1750
 $EndSCHEMATC
