File: GTIA.sch (KiCad schematic (older format))
At the start: 74 parts, among them J2 Video, J202 Diag, J210 Diag, Q1 2N3904, Q2 2N3904, Q3 2N3904, Q6 2N3904, U17 GTIA, U18 74LS08, U20 4050, U21 74LS74, Y2 4,43 MHz

Commit message: Almost finished
Parts:
- FB9: footprint Atari:L_Axial_L7.0mm_D3.3mm_P12.50mm_Horizontal_Fastron_MICC -> Inductor_SMD:L_1812_4532Metric_Pad1.30x3.40mm_HandSolder
- R204, R52, R53: footprint Atari:R_Axial_DIN0207_L3.6mm_D2.2mm_P10.16mm_Horizontal -> Resistor_SMD:R_1206_3216Metric_Pad1.42x1.75mm_HandSolder
Changed lines of the file:
@@
 F 0 "R52" V 8750 2050 50  0000 L CNN
 F 1 "2k" H 8800 2125 50  0000 L CNN
-F 2 "Atari:R_Axial_DIN0207_L3.6mm_D2.2mm_P10.16mm_Horizontal" V 8680 2125 50  0001 C CNN
+F 2 "Resistor_SMD:R_1206_3216Metric_Pad1.42x1.75mm_HandSolder" V 8680 2125 50  0001 C CNN
 F 3 "~" H 8750 2125 50  0001 C CNN
 	1    8750 2125
@@
 F 0 "R53" V 9300 2050 50  0000 L CNN
 F 1 "75" H 9350 2125 50  0000 L CNN
-F 2 "Atari:R_Axial_DIN0207_L3.6mm_D2.2mm_P10.16mm_Horizontal" V 9230 2125 50  0001 C CNN
+F 2 "Resistor_SMD:R_1206_3216Metric_Pad1.42x1.75mm_HandSolder" V 9230 2125 50  0001 C CNN
 F 3 "~" H 9300 2125 50  0001 C CNN
 	1    9300 2125
@@
 F 0 "R204" V 9750 1900 50  0000 C CNN
 F 1 "75" V 9925 1900 50  0000 C CNN
-F 2 "Atari:R_Axial_DIN0207_L3.6mm_D2.2mm_P10.16mm_Horizontal" V 9755 1900 50  0001 C CNN
+F 2 "Resistor_SMD:R_1206_3216Metric_Pad1.42x1.75mm_HandSolder" V 9755 1900 50  0001 C CNN
 F 3 "~" H 9825 1900 50  0001 C CNN
 	1    9825 1900
@@
 F 0 "FB9" V 10100 1925 50  0000 C CNN
 F 1 "Ferrite_Bead" V 10475 1900 50  0000 C CNN
-F 2 "Atari:L_Axial_L7.0mm_D3.3mm_P12.50mm_Horizontal_Fastron_MICC" V 10205 1900 50  0001 C CNN
+F 2 "Inductor_SMD:L_1812_4532Metric_Pad1.30x3.40mm_HandSolder" V 10205 1900 50  0001 C CNN
 F 3 "~" H 10275 1900 50  0001 C CNN
 	1    10275 1900
