File: MMU.sch (KiCad schematic (older format))
At the start: 8 parts, among them U18 74LS08, U2 74LS138, U3 MMU

Commit message: PAL to smd
Parts:
- C26: footprint Atari:C_Axial_L5.1mm_D2.5mm_P12.50mm_Horizontal -> Capacitor_SMD:C_1206_3216Metric_Pad1.42x1.75mm_HandSolder
- R13, R14, R15: footprint Atari:R_Axial_DIN0207_L3.6mm_D2.2mm_P10.16mm_Horizontal -> Resistor_SMD:R_1206_3216Metric_Pad1.42x1.75mm_HandSolder
Changed lines of the file:
@@
 F 0 "R15" H 1545 2071 50  0000 L CNN
 F 1 "3k" H 1545 1980 50  0000 L CNN
-F 2 "Atari:R_Axial_DIN0207_L3.6mm_D2.2mm_P10.16mm_Horizontal" V 1405 2025 50  0001 C CNN
+F 2 "Resistor_SMD:R_1206_3216Metric_Pad1.42x1.75mm_HandSolder" V 1405 2025 50  0001 C CNN
 F 3 "~" H 1475 2025 50  0001 C CNN
 	1    1475 2025
@@
 F 0 "C26" H 4440 5396 50  0000 L CNN
 F 1 "100nF" H 4440 5305 50  0000 L CNN
-F 2 "Atari:C_Axial_L5.1mm_D2.5mm_P12.50mm_Horizontal" H 4363 5200 50  0001 C CNN
+F 2 "Capacitor_SMD:C_1206_3216Metric_Pad1.42x1.75mm_HandSolder" H 4363 5200 50  0001 C CNN
 F 3 "~" H 4325 5350 50  0001 C CNN
 	1    4325 5350
@@
 F 0 "R13" H 2320 2071 50  0000 L CNN
 F 1 "1k" H 2320 1980 50  0000 L CNN
-F 2 "Atari:R_Axial_DIN0207_L3.6mm_D2.2mm_P10.16mm_Horizontal" V 2180 2025 50  0001 C CNN
+F 2 "Resistor_SMD:R_1206_3216Metric_Pad1.42x1.75mm_HandSolder" V 2180 2025 50  0001 C CNN
 F 3 "~" H 2250 2025 50  0001 C CNN
 	1    2250 2025
@@
 F 0 "R14" H 2670 2071 50  0000 L CNN
 F 1 "1k" H 2670 1980 50  0000 L CNN
-F 2 "Atari:R_Axial_DIN0207_L3.6mm_D2.2mm_P10.16mm_Horizontal" V 2530 2025 50  0001 C CNN
+F 2 "Resistor_SMD:R_1206_3216Metric_Pad1.42x1.75mm_HandSolder" V 2530 2025 50  0001 C CNN
 F 3 "~" H 2600 2025 50  0001 C CNN
 	1    2600 2025

Commit message: Almost finished
Parts:
- R12: footprint Atari:R_Axial_DIN0207_L3.6mm_D2.2mm_P10.16mm_Horizontal -> Resistor_SMD:R_1206_3216Metric_Pad1.42x1.75mm_HandSolder
Changed lines of the file:
@@
 F 0 "R12" H 1845 2071 50  0000 L CNN
 F 1 "3k" H 1845 1980 50  0000 L CNN
-F 2 "Atari:R_Axial_DIN0207_L3.6mm_D2.2mm_P10.16mm_Horizontal" V 1705 2025 50  0001 C CNN
+F 2 "Resistor_SMD:R_1206_3216Metric_Pad1.42x1.75mm_HandSolder" V 1705 2025 50  0001 C CNN
 F 3 "~" H 1775 2025 50  0001 C CNN
 	1    1775 2025
