File: Sally_Antic.sch (KiCad schematic (older format))
At the start: 10 parts, among them U18 74LS08, U7 Antic, U8 Sally

Commit message: SMD continue
Parts:
- C31: footprint Atari:C_Axial_L5.1mm_D2.5mm_P12.50mm_Horizontal -> Capacitor_SMD:C_1206_3216Metric_Pad1.42x1.75mm_HandSolder
- R21, R22, R31, R34: footprint Atari:R_Axial_DIN0207_L3.6mm_D2.2mm_P10.16mm_Horizontal -> Resistor_SMD:R_1206_3216Metric_Pad1.42x1.75mm_HandSolder
Changed lines of the file:
@@
 F 0 "C31" H 3190 2321 50  0000 L CNN
 F 1 "100nF" H 3190 2230 50  0000 L CNN
-F 2 "Atari:C_Axial_L5.1mm_D2.5mm_P12.50mm_Horizontal" H 3113 2125 50  0001 C CNN
+F 2 "Capacitor_SMD:C_1206_3216Metric_Pad1.42x1.75mm_HandSolder" H 3113 2125 50  0001 C CNN
 F 3 "~" H 3075 2275 50  0001 C CNN
 	1    3075 2275
@@
 F 0 "R31" H 1995 1571 50  0000 L CNN
 F 1 "3k" H 1995 1480 50  0000 L CNN
-F 2 "Atari:R_Axial_DIN0207_L3.6mm_D2.2mm_P10.16mm_Horizontal" V 1855 1525 50  0001 C CNN
+F 2 "Resistor_SMD:R_1206_3216Metric_Pad1.42x1.75mm_HandSolder" V 1855 1525 50  0001 C CNN
 F 3 "~" H 1925 1525 50  0001 C CNN
 	1    1925 1525
@@
 F 0 "R34" H 1095 1546 50  0000 L CNN
 F 1 "3k" H 1095 1455 50  0000 L CNN
-F 2 "Atari:R_Axial_DIN0207_L3.6mm_D2.2mm_P10.16mm_Horizontal" V 955 1500 50  0001 C CNN
+F 2 "Resistor_SMD:R_1206_3216Metric_Pad1.42x1.75mm_HandSolder" V 955 1500 50  0001 C CNN
 F 3 "~" H 1025 1500 50  0001 C CNN
 	1    1025 1500
@@
 F 0 "R22" H 1395 1571 50  0000 L CNN
 F 1 "3k" H 1395 1480 50  0000 L CNN
-F 2 "Atari:R_Axial_DIN0207_L3.6mm_D2.2mm_P10.16mm_Horizontal" V 1255 1525 50  0001 C CNN
+F 2 "Resistor_SMD:R_1206_3216Metric_Pad1.42x1.75mm_HandSolder" V 1255 1525 50  0001 C CNN
 F 3 "~" H 1325 1525 50  0001 C CNN
 	1    1325 1525
@@
 F 0 "R21" H 1670 1571 50  0000 L CNN
 F 1 "3k" H 1670 1480 50  0000 L CNN
-F 2 "Atari:R_Axial_DIN0207_L3.6mm_D2.2mm_P10.16mm_Horizontal" V 1530 1525 50  0001 C CNN
+F 2 "Resistor_SMD:R_1206_3216Metric_Pad1.42x1.75mm_HandSolder" V 1530 1525 50  0001 C CNN
 F 3 "~" H 1600 1525 50  0001 C CNN
 	1    1600 1525

Commit message: Almost finished
Parts:
- C30: footprint Atari:C_Axial_L5.1mm_D2.5mm_P12.50mm_Horizontal -> Capacitor_SMD:C_1206_3216Metric_Pad1.42x1.75mm_HandSolder
Changed lines of the file:
@@
 F 0 "C30" H 8715 5021 50  0000 L CNN
 F 1 "100nF" H 8715 4930 50  0000 L CNN
-F 2 "Atari:C_Axial_L5.1mm_D2.5mm_P12.50mm_Horizontal" H 8638 4825 50  0001 C CNN
+F 2 "Capacitor_SMD:C_1206_3216Metric_Pad1.42x1.75mm_HandSolder" H 8638 4825 50  0001 C CNN
 F 3 "~" H 8600 4975 50  0001 C CNN
 	1    8600 4975
